File: 0101-INDICATORS.kicad_sch (KiCad schematic)
At the start: 20 parts, among them J1 Conn_02x07_Odd_Even

Commit message: Output SCH
Other:
- company: (none) -> TileParts
- title: #0102 -> #0101 INDICATORS
Changed lines of the file:
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@@
   (paper "A4")
   (title_block
-    (title "#0102")
+    (title "#0101 INDICATORS")
+    (date "2022-10-07")
+    (rev "V1.0")
+    (company "TileParts")
   )
   (junction (at 63.5 106.68) (diameter 0) (color 0 0 0 0)
